Commit message: Working moveit config for centauro kairos

File: centauro_rbkairos_plus_moveit_config/config/centauro_rbkairos_plus.ros2_control.xacro (robot description, xacro)
@@ -1,5 +1,5 @@
 <?xml version="1.0"?>
 <robot xmlns:xacro="http://www.ros.org/wiki/xacro">
-    <xacro:macro name="rbkairos_plus_ros2_control" params="name initial_positions_file">
+    <xacro:macro name="centauro_rbkairos_plus_ros2_control" params="name initial_positions_file">
         <xacro:property name="initial_positions" value="${xacro.load_yaml(initial_positions_file)['initial_positions']}"/>
         <ros2_control name="${name}" type="system">
